File: qomu-board.kicad_pcb (KiCad board)
At the start: 6 copper layers, 28.1 x 10.7 mm, 61 parts, among them IC1 EOS-S3, J1 FTSH-105-01-L-DV-K, J2 825437-4, J3 22-23-2021, Q1 RV1C002UN, Q2 RV1C002UN, Q3 RV1C002UN, SW2 Captouch Pads, U1 MIC5504-3.3YMT, U10 UHD1110-FKA, U2 MIC5504-3.3YMT, U4 GD25Q16CEIGR, U5 MC3635, U9 USB-B

Commit message: Edited tech notes on PCB
Other:
- board text added: "PCB Thickness: 0.6mm"
- board text removed: "PCB Soldermask: Dark Blue PCB Thickness: 0.6mm Hard gold plating on fingers, side ENIG on other surfaces"
Changed lines of the file:
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@@
     (4 In4.Cu signal)
     (31 Bottom signal)
-    (32 B.Adhes user hide)
-    (33 F.Adhes user hide)
-    (34 B.Paste user hide)
-    (35 F.Paste user hide)
+    (32 B.Adhes user)
+    (33 F.Adhes user)
+    (34 B.Paste user)
+    (35 F.Paste user)
     (36 B.SilkS user)
-    (37 F.SilkS user hide)
+    (37 F.SilkS user)
     (38 B.Mask user)
-    (39 F.Mask user hide)
-    (40 Dwgs.User user hide)
-    (41 Cmts.User user hide)
-    (42 Eco1.User user hide)
-    (43 Eco2.User user hide)
+    (39 F.Mask user)
+    (40 Dwgs.User user)
+    (41 Cmts.User user)
+    (42 Eco1.User user)
+    (43 Eco2.User user)
     (44 Edge.Cuts user)
-    (45 Margin user hide)
+    (45 Margin user)
     (46 B.CrtYd user)
-    (47 F.CrtYd user hide)
-    (48 B.Fab user hide)
-    (49 F.Fab user hide)
+    (47 F.CrtYd user)
+    (48 B.Fab user)
+    (49 F.Fab user)
   )
   (setup
-    (last_trace_width 0.2)
+    (last_trace_width 0.1)
     (user_trace_width 0.1)
     (user_trace_width 0.15)
@@
   (gr_arc (start 21.393939 18.205) (end 20.91697 18.355) (angle -72.54239688) (layer Cmts.User) (width 0.1))
   (gr_arc (start 20.44 18.505) (end 21.203151 18.265) (angle -72.54239689) (layer Cmts.User) (width 0.1))
-  (gr_text "PCB Soldermask: Dark Blue\nPCB Thickness: 0.6mm\nHard gold plating on fingers, side\nENIG on other surfaces" (at 16.55 37.45) (layer Eco1.User)
+  (gr_text "PCB Thickness: 0.6mm" (at 16.55 37.45) (layer Eco1.User)
     (effects (font (size 2.5 2.5) (thickness 0.3)) (justify left))
   )
@@
   (via micro (at 17.38 25.76) (size 0.3) (drill 0.15) (layers GND.Cu In4.Cu) (net 1))
   (via micro (at 17.37 25.409) (size 0.3) (drill 0.15) (layers In4.Cu Bottom) (net 1))
-  (via (at 25.07 24.41) (size 0.3) (drill 0.15) (layers Top Bottom) (net 26))
-  (via (at 18.91 24.6) (size 0.3) (drill 0.15) (layers Top Bottom) (net 26))
-  (via micro (at 25.86 26.08) (size 0.3) (drill 0.15) (layers GND.Cu In4.Cu) (net 2))
-  (via micro (at 26.26 26.08) (size 0.3) (drill 0.15) (layers In2.Cu GND.Cu) (net 2))
-  (via micro (at 25.47 26.08) (size 0.3) (drill 0.15) (layers In4.Cu Bottom) (net 2))
   (via (at 22.09 19.449) (size 0.35) (drill 0.15) (layers Top Bottom) (net 1))
   (via (at 17.36 18.729) (size 0.35) (drill 0.15) (layers Top Bottom) (net 1))
@@
   (segment (start 21.831793 19.707207) (end 21.831793 20.848207) (width 0.4) (layer In4.Cu) (net 1))
   (segment (start 27.45 18.659) (end 26.399 18.659) (width 0.2) (layer GND.Cu) (net 1))
+  (via micro (at 25.86 26.08) (size 0.3) (drill 0.15) (layers GND.Cu In4.Cu) (net 2))
+  (via micro (at 26.26 26.08) (size 0.3) (drill 0.15) (layers In2.Cu GND.Cu) (net 2))
+  (via micro (at 25.47 26.08) (size 0.3) (drill 0.15) (layers In4.Cu Bottom) (net 2))
   (via micro (at 22.82 22.629) (size 0.3) (drill 0.15) (layers In4.Cu Bottom) (net 2))
   (via micro (at 19.79 24.209) (size 0.3) (drill 0.15) (layers GND.Cu In4.Cu) (net 2))
@@
   (segment (start 22.21 17.7008) (end 21.22 18.6908) (width 0.1) (layer Bottom) (net 25))
   (segment (start 21.22 18.6908) (end 21.22 19.939) (width 0.1) (layer Bottom) (net 25))
+  (via (at 25.07 24.41) (size 0.3) (drill 0.15) (layers Top Bottom) (net 26))
+  (via (at 18.91 24.6) (size 0.3) (drill 0.15) (layers Top Bottom) (net 26))
   (via (at 25.43 24.189) (size 0.3) (drill 0.15) (layers Top Bottom) (net 26))
   (segment (start 17.81 24.919) (end 17.38 24.919) (width 0.15) (layer Bottom) (net 26))
