File: qomu-board.sch (KiCad schematic (older format))
At the start: 51 parts, among them IC1 EOS-S3, J1 FTSH-105-01-L-DV-K, J2 825437-4, Q1 RV1C002UN, Q2 RV1C002UN, Q3 RV1C002UN, SW2 Captouch Pads, U1 MIC5504-3.3YMT, U10 UHD1110-FKA, U2 MIC5504-3.3YMT, U4 GD25Q16CEIGR, U5 MC3635, U9 USB-B

Commit message: Removed R6 and R7
Parts:
- removed R6, R7: 10k, qomu-board-footprints:R_0201_0603Metric, symbol qomu-board:R_10k_0201
Connections:
- wire segments 225 -> 217
- no-connect marks 9 -> 11
Changed lines of the file:
@@
 	3550 3250 4100 3250
-$Comp
-L qomu-board:R_10k_0201 R7
-U 1 1 5DDFBEAE
-P 3850 4150
-F 0 "R7" V 3800 4000 50  0000 C CNN
-F 1 "10k" V 3800 4300 50  0000 C CNN
-F 2 "qomu-board-footprints:R_0201_0603Metric" H 3850 4150 50  0001 C CNN
-F 3 "" H 3850 4150 50  0001 C CNN
-F 4 "ERJ1GNF1002C " H -4900 2450 50  0001 C CNN "MPN"
-F 5 "Panasonic" H 0   0   50  0001 C CNN "Manufacturer"
-	1    3850 4150
-	0    1    1    0
-$EndComp
-$Comp
-L qomu-board:R_10k_0201 R6
-U 1 1 5DDFBEB5
-P 3850 4050
-F 0 "R6" V 3900 4200 50  0000 C CNN
-F 1 "10k" V 3900 3900 50  0000 C CNN
-F 2 "qomu-board-footprints:R_0201_0603Metric" H 3850 4050 50  0001 C CNN
-F 3 "" H 3850 4050 50  0001 C CNN
-F 4 "ERJ1GNF1002C " H -4900 2350 50  0001 C CNN "MPN"
-F 5 "Panasonic" H 0   0   50  0001 C CNN "Manufacturer"
-	1    3850 4050
-	0    -1   -1   0
-$EndComp
-Wire Wire Line
-	3550 4050 3650 4050
-Wire Wire Line
-	3550 4150 3750 4150
-Wire Wire Line
-	3950 4050 4300 4050
-Wire Wire Line
-	4300 4050 4300 4150
-Wire Wire Line
-	4300 4150 3950 4150
-Wire Wire Line
-	4300 4150 4300 4300
-Connection ~ 4300 4150
-$Comp
-L qomu-board:GND #PWR015
-U 1 1 5DE27F69
-P 4300 4300
-F 0 "#PWR015" H 4300 4050 50  0001 C CNN
-F 1 "GND" H 4305 4127 50  0000 C CNN
-F 2 "" H 4300 4300 50  0001 C CNN
-F 3 "" H 4300 4300 50  0001 C CNN
-	1    4300 4300
-	1    0    0    -1
-$EndComp
 $Comp
 L qomu-board:GND #PWR014
@@
 Text Label 3650 2950 0    50   ~ 0
 SWD_CLK
-Wire Wire Line
-	3650 4050 3650 3950
-Wire Wire Line
-	3650 3950 3950 3950
-Connection ~ 3650 4050
-Wire Wire Line
-	3650 4050 3750 4050
-Text Label 3650 3950 0    50   ~ 0
+Text Label 3650 4050 0    50   ~ 0
 DBG_SS
 Wire Wire Line
@@
 Wire Wire Line
 	3550 3050 3950 3050
+Wire Wire Line
+	3550 4050 4000 4050
+NoConn ~ 3550 4150
+NoConn ~ 3550 3850
 $EndSCHEMATC

Commit message: Removed DBG_SS signal
Parts:
- removed R10: 10k, qomu-board-footprints:R_0201_0603Metric, symbol qomu-board:R_10k_0201
- removed R14: R_0R_0402, qomu-board-footprints:0402-res, symbol qomu-board:R_0R_0402
Connections:
- net labels removed: DBG_SS
- wire segments 217 -> 210
- no-connect marks 11 -> 14
Other:
- note removed: "DNP"
Changed lines of the file:
@@
 	5950 5100 7400 5100
 Wire Wire Line
-	5950 4900 6100 4900
-Wire Wire Line
-	6700 4900 7400 4900
-Text Notes 6700 4900 0    50   ~ 10
-DNP
-Wire Wire Line
 	5950 4800 6400 4800
 Wire Wire Line
 	5950 4700 6700 4700
-Wire Wire Line
-	6100 4650 6100 4900
-Connection ~ 6100 4900
-Wire Wire Line
-	6100 4900 6400 4900
 Wire Wire Line
 	6400 4650 6400 4800
@@
 Text Label 7000 4800 0    50   ~ 0
 SWD_CLK
-Text Label 7000 4900 0    50   ~ 0
-DBG_SS
 Wire Wire Line
 	6950 5950 6800 5950
@@
 $EndComp
 $Comp
-L qomu-board:R_0R_0402 R14
-U 1 1 5DED5709
-P 6550 4900
-F 0 "R14" H 6250 4950 60  0000 C CNN
-F 1 "R_0R_0402" H 6550 4750 60  0001 C CNN
-F 2 "qomu-board-footprints:0402-res" H 6750 5100 60  0001 L CNN
-F 3 "" H 6550 4900 50  0001 C CNN
-F 4 "PANASONIC" H 6750 5300 60  0001 L CNN "Manufacturer"
-F 5 "ERJ2GE0R00X" H 6750 5200 60  0001 L CNN "MPN"
-F 6 "0R" H 6250 4850 50  0000 C CNN "Val"
-	1    6550 4900
-	1    0    0    -1
-$EndComp
-$Comp
 L qomu-board:FTSH-105-01-L-DV-K J1
 U 1 1 5DED6D58
@@
 	-1   0    0    1
 $EndComp
-$Comp
-L qomu-board:R_10k_0201 R10
-U 1 1 5DEA75F7
-P 6100 4550
-F 0 "R10" H 6150 4450 50  0000 C CNN
-F 1 "10k" V 6000 4550 50  0000 C CNN
-F 2 "qomu-board-footprints:R_0201_0603Metric" H 6100 4550 50  0001 C CNN
-F 3 "" H 6100 4550 50  0001 C CNN
-F 4 "ERJ1GNF1002C " H -2650 2850 50  0001 C CNN "MPN"
-F 5 "Panasonic" H 0   0   50  0001 C CNN "Manufacturer"
-	1    6100 4550
-	-1   0    0    1
-$EndComp
-Wire Wire Line
-	6100 4450 6100 4400
-Wire Wire Line
-	6100 4400 6400 4400
 Wire Wire Line
 	6700 4400 6700 4450
@@
 Text Label 3650 2950 0    50   ~ 0
 SWD_CLK
-Text Label 3650 4050 0    50   ~ 0
-DBG_SS
 Wire Wire Line
 	3550 5450 4000 5450
@@
 Wire Wire Line
 	3550 3050 3950 3050
-Wire Wire Line
-	3550 4050 4000 4050
 NoConn ~ 3550 4150
 NoConn ~ 3550 3850
+NoConn ~ 5950 4900
+NoConn ~ 3550 3950
+NoConn ~ 3550 4050
 $EndSCHEMATC

Commit message: Updated PDF with schematic, updated BOM
Parts:
- added J3: 22-23-2021, antmicro-footprints:PinHeader_1x2_P2.54mm_Drill1.02mm, symbol qomu-board:22-23-2021
- added R6: 10k, qomu-board-footprints:R_0201_0603Metric, symbol qomu-board:R_10k_0201
- D1, D2, D3, D4, D6, D7: footprint qomu-board:X1-DFN1006-2 -> qomu-board-footprints:X1-DFN1006-2
- D5: footprint qomu-board:TVS-11V -> qomu-board-footprints:X1-DFN1006-2
- U1, U2: footprint qomu-board:Texas_X2SON-4_1x1mm_P0.65mm -> qomu-board-footprints:Texas_X2SON-4_1x1mm_P0.65mm
- U10: footprint qomu-board:LED-RGB-5DS-UHD1110-FKA -> qomu-board-footprints:LED-RGB-5DS-UHD1110-FKA
Connections:
- wire segments 210 -> 214
- no-connect marks 14 -> 13
Other:
- note removed: "Currently not connected"
Changed lines of the file:
@@
 F 0 "U10" H 8400 2900 50  0000 C CNN
 F 1 "UHD1110-FKA" H 8600 2800 50  0000 C CNN
-F 2 "qomu-board:LED-RGB-5DS-UHD1110-FKA" H 8600 2950 50  0001 C CNN
+F 2 "qomu-board-footprints:LED-RGB-5DS-UHD1110-FKA" H 8600 2950 50  0001 C CNN
 F 3 "https://www.cree.com/led-components/media/documents/ds-UHD1110-FKA.pdf" H 8600 2950 50  0001 C CNN
 F 4 "UHD1110-FKA" H 8600 2950 50  0001 C CNN "MPN"
@@
 F 0 "D1" V 5950 1600 50  0000 L CNN
 F 1 "D5V0L1B2LP3-7" H 6000 1800 50  0001 L CNN
-F 2 "qomu-board:X1-DFN1006-2" V 6050 1700 50  0001 C CNN
+F 2 "qomu-board-footprints:X1-DFN1006-2" V 6050 1700 50  0001 C CNN
 F 3 "https://www.diodes.com/assets/Datasheets/D5V0L1B2LP3.pdf" V 6050 1700 50  0001 C CNN
 F 4 "Diodes Inc." V 6050 1700 50  0001 C CNN "Manufacturer"
@@
 F 0 "D2" V 6250 1600 50  0000 L CNN
 F 1 "D5V0L1B2LP3-7" H 6300 1800 50  0001 L CNN
-F 2 "qomu-board:X1-DFN1006-2" V 6350 1700 50  0001 C CNN
+F 2 "qomu-board-footprints:X1-DFN1006-2" V 6350 1700 50  0001 C CNN
 F 3 "https://www.diodes.com/assets/Datasheets/D5V0L1B2LP3.pdf" V 6350 1700 50  0001 C CNN
 F 4 "Diodes Inc." V 6350 1700 50  0001 C CNN "Manufacturer"
@@
 F 0 "D3" V 6100 1600 50  0000 L CNN
 F 1 "D5V0L1B2LP3-7" H 6150 1800 50  0001 L CNN
-F 2 "qomu-board:X1-DFN1006-2" V 6200 1700 50  0001 C CNN
+F 2 "qomu-board-footprints:X1-DFN1006-2" V 6200 1700 50  0001 C CNN
 F 3 "https://www.diodes.com/assets/Datasheets/D5V0L1B2LP3.pdf" V 6200 1700 50  0001 C CNN
 F 4 "Diodes Inc." V 6200 1700 50  0001 C CNN "Manufacturer"
@@
 F 0 "D4" V 6400 1600 50  0000 L CNN
 F 1 "D5V0L1B2LP3-7" V 6600 600 50  0000 L CNN
-F 2 "qomu-board:X1-DFN1006-2" V 6500 1700 50  0001 C CNN
+F 2 "qomu-board-footprints:X1-DFN1006-2" V 6500 1700 50  0001 C CNN
 F 3 "https://www.diodes.com/assets/Datasheets/D5V0L1B2LP3.pdf" V 6500 1700 50  0001 C CNN
 F 4 "Diodes Inc." V 6500 1700 50  0001 C CNN "Manufacturer"
@@
 F 0 "D6" V 9500 1500 50  0000 L CNN
 F 1 "D5V0L1B2LP3-7" V 9500 550 50  0000 L CNN
-F 2 "qomu-board:X1-DFN1006-2" V 9500 1450 50  0001 C CNN
+F 2 "qomu-board-footprints:X1-DFN1006-2" V 9500 1450 50  0001 C CNN
 F 3 "https://www.diodes.com/assets/Datasheets/D5V0L1B2LP3.pdf" V 9500 1450 50  0001 C CNN
 F 4 "Diodes Inc." V 9500 1450 50  0001 C CNN "Manufacturer"
@@
 F 0 "D7" V 9600 1300 50  0000 L CNN
 F 1 "D5V0L1B2LP3-7" V 9500 650 50  0000 L CNN
-F 2 "qomu-board:X1-DFN1006-2" V 9600 1450 50  0001 C CNN
+F 2 "qomu-board-footprints:X1-DFN1006-2" V 9600 1450 50  0001 C CNN
 F 3 "https://www.diodes.com/assets/Datasheets/D5V0L1B2LP3.pdf" V 9600 1450 50  0001 C CNN
 F 4 "Diodes Inc." V 9600 1450 50  0001 C CNN "Manufacturer"
@@
 F 0 "D5" H 9300 1450 50  0000 L CNN
 F 1 "VCUT05E1-SD0" H 9300 1350 50  0000 L CNN
-F 2 "qomu-board:TVS-11V" V 9350 1250 50  0001 C CNN
+F 2 "qomu-board-footprints:X1-DFN1006-2" V 9350 1250 50  0001 C CNN
 F 3 "http://www.vishay.com/docs/85900/vcut05e1-sd0.pdf" V 9350 1250 50  0001 C CNN
 F 4 "Diodes Inc." V 9350 1250 50  0001 C CNN "Manufacturer"
@@
 F 0 "U2" H 1750 1700 50  0000 C CNN
 F 1 "MIC5504-3.3YMT" H 2000 1600 50  0000 C CNN
-F 2 "qomu-board:Texas_X2SON-4_1x1mm_P0.65mm" H 1900 1200 50  0001 C CNN
+F 2 "qomu-board-footprints:Texas_X2SON-4_1x1mm_P0.65mm" H 1900 1200 50  0001 C CNN
 F 3 "" H 1900 1200 50  0001 C CNN
 F 4 "MIC5504-3.3YMT" H 250 -100 50  0001 C CNN "MPN"
@@
 F 0 "U1" H 1750 1650 50  0000 C CNN
 F 1 "MIC5504-3.3YMT" H 2000 1550 50  0000 C CNN
-F 2 "qomu-board:Texas_X2SON-4_1x1mm_P0.65mm" H 1900 1700 50  0001 C CNN
+F 2 "qomu-board-footprints:Texas_X2SON-4_1x1mm_P0.65mm" H 1900 1700 50  0001 C CNN
 F 3 "" H 1900 1700 50  0001 C CNN
 F 4 "MIC5504-3.3YMT" H 250 400 50  0001 C CNN "MPN"
@@
 Wire Wire Line
 	5600 1450 6200 1450
-Text Notes 5950 1000 0    50   ~ 0
-Currently not connected
 Wire Wire Line
 	4300 3150 4300 3250
@@
 Wire Wire Line
 	3550 3050 3950 3050
-NoConn ~ 3550 4150
 NoConn ~ 3550 3850
 NoConn ~ 5950 4900
 NoConn ~ 3550 3950
 NoConn ~ 3550 4050
+$Comp
+L qomu-board:22-23-2021 J3
+U 1 1 5E147536
+P 4300 3700
+F 0 "J3" H 4600 3750 50  0000 R CNN
+F 1 "22-23-2021" H 4900 3850 50  0000 R CNN
+F 2 "antmicro-footprints:PinHeader_1x2_P2.54mm_Drill1.02mm" H 4500 3900 60  0001 L CNN
+F 3 "https://media.digikey.com/pdf/Data%20Sheets/Molex%20PDFs/A-6373-N_Series_Dwg_2010-12-03.pdf" H 4500 4000 60  0001 L CNN
+F 4 "22-23-2021" H 4500 4200 60  0001 L CNN "MPN"
+F 5 "Molex" H 4500 4800 60  0001 L CNN "Manufacturer"
+	1    4300 3700
+	-1   0    0    1
+$EndComp
+$Comp
+L qomu-board:R_10k_0201 R6
+U 1 1 5E151CF7
+P 4100 4000
+F 0 "R6" V 4150 4200 50  0000 C CNN
+F 1 "10k" V 4000 4000 50  0000 C CNN
+F 2 "qomu-board-footprints:R_0201_0603Metric" H 4100 4000 50  0001 C CNN
+F 3 "" H 4100 4000 50  0001 C CNN
+F 4 "ERJ1GNF1002C " H -4650 2300 50  0001 C CNN "MPN"
+F 5 "Panasonic" H -2300 -550 50  0001 C CNN "Manufacturer"
+	1    4100 4000
+	0    -1   -1   0
+$EndComp
+$Comp
+L qomu-board:+3V3 #PWR011
+U 1 1 5E1531DB
+P 4350 3800
+F 0 "#PWR011" H 4350 3800 50  0001 C CNN
+F 1 "+3V3" V 4450 3750 50  0000 C CNN
+F 2 "" H 4350 3800 50  0001 C CNN
+F 3 "" H 4350 3800 50  0001 C CNN
+	1    4350 3800
+	0    1    1    0
+$EndComp
+Wire Wire Line
+	3550 4150 3850 4150
+Wire Wire Line
+	3850 4150 3850 4000
+Wire Wire Line
+	4200 4000 4200 3800
+Wire Wire Line
+	3850 4000 4000 4000
 $EndSCHEMATC

Commit message: Added oscillator, updated component placement
Parts:
- added C13, C14: 8p, qomu-board-footprints:C_0201_0603Metric, symbol qomu-board:C_8p_0201
- added XTAL1: ECS-_327-12_5-1210-TR, qomu-board-footprints:XTAL_ECS-.327-12.5-1210-TR, symbol qomu-board:ECS-_327-12_5-1210-TR
- J3: footprint antmicro-footprints:PinHeader_1x2_P2.54mm_Drill1.02mm -> qomu-board-footprints:PinHeader_1x2_P2.54mm_Drill1.02mm
Connections:
- wire segments 214 -> 219
- no-connect marks 13 -> 11
Changed lines of the file:
@@
 EESchema Schematic File Version 4
+LIBS:qomu-board-cache
 EELAYER 30 0
 EELAYER END
@@
 NoConn ~ 1500 3450
 NoConn ~ 1500 3550
-NoConn ~ 1500 3850
-NoConn ~ 1500 3950
 NoConn ~ 1500 4100
 $Comp
@@
 F 0 "J3" H 4600 3750 50  0000 R CNN
 F 1 "22-23-2021" H 4900 3850 50  0000 R CNN
-F 2 "antmicro-footprints:PinHeader_1x2_P2.54mm_Drill1.02mm" H 4500 3900 60  0001 L CNN
+F 2 "qomu-board-footprints:PinHeader_1x2_P2.54mm_Drill1.02mm" H 4500 3900 60  0001 L CNN
 F 3 "https://media.digikey.com/pdf/Data%20Sheets/Molex%20PDFs/A-6373-N_Series_Dwg_2010-12-03.pdf" H 4500 4000 60  0001 L CNN
 F 4 "22-23-2021" H 4500 4200 60  0001 L CNN "MPN"
@@
 Wire Wire Line
 	3850 4000 4000 4000
+$Comp
+L qomu-board:C_8p_0201 C14
+U 1 1 5E00A59A
+P 1100 4100
+F 0 "C14" H 1201 4146 50  0000 L CNN
+F 1 "8p" H 1201 4055 50  0000 L CNN
+F 2 "qomu-board-footprints:C_0201_0603Metric" H 1256 4494 50  0001 C CNN
+F 3 "" H 1100 4100 50  0001 C CNN
+F 4 "Murata" H 1112 4654 50  0001 C CNN "Manufacturer"
+F 5 "GRM0335C1E8R0DA01D" H 1132 4578 50  0001 C CNN "MPN"
+	1    1100 4100
+	1    0    0    -1
+$EndComp
+$Comp
+L qomu-board:C_8p_0201 C13
+U 1 1 5E00BE50
+P 800 4100
+F 0 "C13" H 901 4146 50  0000 L CNN
+F 1 "8p" H 901 4055 50  0000 L CNN
+F 2 "qomu-board-footprints:C_0201_0603Metric" H 956 4494 50  0001 C CNN
+F 3 "" H 800 4100 50  0001 C CNN
+F 4 "Murata" H 812 4654 50  0001 C CNN "Manufacturer"
+F 5 "GRM0335C1E8R0DA01D" H 832 4578 50  0001 C CNN "MPN"
+	1    800  4100
+	1    0    0    -1
+$EndComp
+Wire Wire Line
+	1500 3850 1100 3850
+Wire Wire Line
+	800  3950 800  3850
+Wire Wire Line
+	800  3950 800  4000
+Connection ~ 800  3950
+Wire Wire Line
+	1500 3950 800  3950
+Wire Wire Line
+	1100 3850 1100 4000
+Connection ~ 1100 3850
+$Comp
+L qomu-board:ECS-_327-12_5-1210-TR XTAL1
+U 1 1 5DFFBEFA
+P 950 3850
+F 0 "XTAL1" H 1250 3900 50  0000 C CNN
+F 1 "ECS-_327-12_5-1210-TR" V 693 3450 50  0000 C CNN
+F 2 "qomu-board-footprints:XTAL_ECS-.327-12.5-1210-TR" H 1150 4050 60  0001 L CNN
+F 3 "https://ecsxtal.com/store/pdf/ECX-1210.pdf" H 1150 4150 60  0001 L CNN
+F 4 "ECS-.327-12.5-1210-TR" H 1158 4224 60  0001 L CNN "MPN"
+F 5 "ECS Inc." H 1174 4302 60  0001 L CNN "Manufacturer"
+	1    950  3850
+	1    0    0    -1
+$EndComp
+$Comp
+L qomu-board:GND #PWR0129
+U 1 1 5E06B803
+P 800 4200
+F 0 "#PWR0129" H 800 3950 50  0001 C CNN
+F 1 "GND" H 805 4027 50  0000 C CNN
+F 2 "" H 800 4200 50  0001 C CNN
+F 3 "" H 800 4200 50  0001 C CNN
+	1    800  4200
+	1    0    0    -1
+$EndComp
+$Comp
+L qomu-board:GND #PWR0130
+U 1 1 5E06BB21
+P 1100 4200
+F 0 "#PWR0130" H 1100 3950 50  0001 C CNN
+F 1 "GND" H 1105 4027 50  0000 C CNN
+F 2 "" H 1100 4200 50  0001 C CNN
+F 3 "" H 1100 4200 50  0001 C CNN
+	1    1100 4200
+	1    0    0    -1
+$EndComp
 $EndSCHEMATC

Commit message: TOUCHx connection changed
Connections:
- wire segments 219 -> 221
- no-connect marks 11 -> 9
Changed lines of the file:
@@
 Wire Wire Line
 	7950 4700 8400 4700
-NoConn ~ 3550 4850
-NoConn ~ 3550 5350
 Wire Wire Line
 	750  3250 1500 3250
@@
 Text Label 3650 3050 0    50   ~ 0
 TOUCH_1
-Text Label 3650 3150 0    50   ~ 0
+Text Label 3650 3350 0    50   ~ 0
 TOUCH_2
-Text Label 3650 3250 0    50   ~ 0
+Text Label 3650 5350 0    50   ~ 0
 TOUCH_3
-Text Label 3650 3350 0    50   ~ 0
+Text Label 3650 4850 0    50   ~ 0
 TOUCH_4
 Wire Wire Line
@@
 	1    0    0    -1
 $EndComp
+Wire Wire Line
+	3550 5350 4000 5350
+Wire Wire Line
+	3550 4850 4000 4850
 $EndSCHEMATC

Commit message: Added testpoints to PCB
Parts:
- added TP1, TP2, TP3, TP4, TP5, TP6, TP7, TP8: TP_SMD_0_75MM, qomu-board-footprints:Testpoint_smd_0_75mm, symbol qomu-board:TP_SMD_0_75MM
Connections:
- net labels added: C1
- wire segments 221 -> 229
- no-connect marks 9 -> 8
Changed lines of the file:
@@
 	1350 2850 1100 2850
 Wire Wire Line
-	1500 3700 1100 3700
+	1500 3700 1300 3700
 Text Label 1000 3700 2    50   ~ 0
 RST_N
@@
 $EndComp
 Wire Wire Line
-	5700 3200 5050 3200
-Wire Wire Line
-	5700 3300 5050 3300
-Wire Wire Line
-	5700 2850 5050 2850
-Wire Wire Line
-	6650 2850 7100 2850
+	5700 3200 5450 3200
+Wire Wire Line
+	5700 3300 5450 3300
+Wire Wire Line
+	5700 2850 5450 2850
+Wire Wire Line
+	6650 2850 6700 2850
 Wire Wire Line
 	6650 3300 6650 3400
@@
 R_USB_P
 Wire Wire Line
-	3550 4250 4200 4250
-Wire Wire Line
 	3550 4550 4000 4550
 Text Label 3650 4250 0    50   ~ 0
@@
 Wire Notes Line
 	600  2300 4450 2300
-Wire Notes Line
-	4450 2300 4450 7700
 Wire Notes Line
 	4450 7700 600  7700
@@
 Wire Wire Line
 	3550 3450 3950 3450
-Text Notes 5450 3600 0    50   ~ 0
+Text Notes 5800 3600 0    50   ~ 0
 operating current\nmax. 20mA
 Text Notes 650  5950 0    50   ~ 0
@@
 Wire Wire Line
 	4300 3250 4300 3350
-$Comp
-L qomu-board:EOS-S3 IC1
-U 1 1 5DCB0652
-P 1600 2700
-F 0 "IC1" H 1650 2850 50  0000 C CNN
-F 1 "EOS-S3" H 1750 2750 50  0000 C CNN
-F 2 "qomu-board:42-WLCSP" H 3250 -400 50  0001 C CNN
-F 3 "https://dev.antmicro.com/attachments/download/9063/ql-eos-s3-datasheet.pdf" H 3350 -300 50  0001 C CNN
-	1    1600 2700
-	1    0    0    -1
-$EndComp
 Text Label 3650 3050 0    50   ~ 0
 TOUCH_1
@@
 Wire Wire Line
 	3550 3050 3950 3050
-NoConn ~ 3550 3850
 NoConn ~ 5950 4900
 NoConn ~ 3550 3950
@@
 L qomu-board:22-23-2021 J3
 U 1 1 5E147536
-P 4300 3700
-F 0 "J3" H 4600 3750 50  0000 R CNN
-F 1 "22-23-2021" H 4900 3850 50  0000 R CNN
-F 2 "qomu-board-footprints:PinHeader_1x2_P2.54mm_Drill1.02mm" H 4500 3900 60  0001 L CNN
-F 3 "https://media.digikey.com/pdf/Data%20Sheets/Molex%20PDFs/A-6373-N_Series_Dwg_2010-12-03.pdf" H 4500 4000 60  0001 L CNN
-F 4 "22-23-2021" H 4500 4200 60  0001 L CNN "MPN"
-F 5 "Molex" H 4500 4800 60  0001 L CNN "Manufacturer"
-	1    4300 3700
-	-1   0    0    1
+P 4900 5750
+F 0 "J3" V 4750 5750 50  0000 R CNN
+F 1 "22-23-2021" V 5100 6050 50  0000 R CNN
+F 2 "qomu-board-footprints:PinHeader_1x2_P2.54mm_Drill1.02mm" H 5100 5950 60  0001 L CNN
+F 3 "https://media.digikey.com/pdf/Data%20Sheets/Molex%20PDFs/A-6373-N_Series_Dwg_2010-12-03.pdf" H 5100 6050 60  0001 L CNN
+F 4 "22-23-2021" H 5100 6250 60  0001 L CNN "MPN"
+F 5 "Molex" H 5100 6850 60  0001 L CNN "Manufacturer"
+	1    4900 5750
+	0    1    1    0
 $EndComp
 $Comp
 L qomu-board:R_10k_0201 R6
 U 1 1 5E151CF7
-P 4100 4000
-F 0 "R6" V 4150 4200 50  0000 C CNN
-F 1 "10k" V 4000 4000 50  0000 C CNN
-F 2 "qomu-board-footprints:R_0201_0603Metric" H 4100 4000 50  0001 C CNN
-F 3 "" H 4100 4000 50  0001 C CNN
-F 4 "ERJ1GNF1002C " H -4650 2300 50  0001 C CNN "MPN"
-F 5 "Panasonic" H -2300 -550 50  0001 C CNN "Manufacturer"
-	1    4100 4000
-	0    -1   -1   0
+P 5350 5850
+F 0 "R6" V 5250 5850 50  0000 C CNN
+F 1 "10k" V 5450 5850 50  0000 C CNN
+F 2 "qomu-board-footprints:R_0201_0603Metric" H 5350 5850 50  0001 C CNN
+F 3 "" H 5350 5850 50  0001 C CNN
+F 4 "ERJ1GNF1002C " H -3400 4150 50  0001 C CNN "MPN"
+F 5 "Panasonic" H -1050 1300 50  0001 C CNN "Manufacturer"
+	1    5350 5850
+	0    1    1    0
 $EndComp
 $Comp
 L qomu-board:+3V3 #PWR011
 U 1 1 5E1531DB
-P 4350 3800
-F 0 "#PWR011" H 4350 3800 50  0001 C CNN
-F 1 "+3V3" V 4450 3750 50  0000 C CNN
-F 2 "" H 4350 3800 50  0001 C CNN
-F 3 "" H 4350 3800 50  0001 C CNN
-	1    4350 3800
-	0    1    1    0
-$EndComp
-Wire Wire Line
-	3550 4150 3850 4150
-Wire Wire Line
-	3850 4150 3850 4000
-Wire Wire Line
-	4200 4000 4200 3800
-Wire Wire Line
-	3850 4000 4000 4000
+P 5050 5650
+F 0 "#PWR011" H 5050 5650 50  0001 C CNN
+F 1 "+3V3" H 5200 5650 50  0000 C CNN
+F 2 "" H 5050 5650 50  0001 C CNN
+F 3 "" H 5050 5650 50  0001 C CNN
+	1    5050 5650
+	1    0    0    -1
+$EndComp
 $Comp
 L qomu-board:C_8p_0201 C14
@@
 Wire Wire Line
 	3550 4850 4000 4850
+$Comp
+L qomu-board:TP_SMD_0_75MM TP2
+U 1 1 5E378204
+P 4100 3850
+F 0 "TP2" V 4100 3800 50  0000 R CNN
+F 1 "TP_SMD_0_75MM" H 4100 3750 50  0001 C CNN
+F 2 "qomu-board-footprints:Testpoint_smd_0_75mm" H 4300 4050 60  0001 L CNN
+F 3 "" H 4300 4150 60  0001 L CNN
+	1    4100 3850
+	0    -1   -1   0
+$EndComp
+$Comp
+L qomu-board:EOS-S3 IC1
+U 1 1 5DCB0652
+P 1600 2700
+F 0 "IC1" H 1650 2850 50  0000 C CNN
+F 1 "EOS-S3" H 1750 2750 50  0000 C CNN
+F 2 "qomu-board:42-WLCSP" H 3250 -400 50  0001 C CNN
+F 3 "https://dev.antmicro.com/attachments/download/9063/ql-eos-s3-datasheet.pdf" H 3350 -300 50  0001 C CNN
+	1    1600 2700
+	1    0    0    -1
+$EndComp
+Wire Wire Line
+	5000 5750 5050 5750
+Wire Wire Line
+	5050 5750 5050 5700
+Wire Wire Line
+	5450 5850 5850 5850
+Wire Wire Line
+	5250 5850 5000 5850
+Wire Wire Line
+	3550 4150 4000 4150
+Wire Wire Line
+	3550 4250 4200 4250
+Text Label 3650 4150 0    50   ~ 0
+C1
+Text Label 5700 5850 0    50   ~ 0
+C1
+Wire Wire Line
+	3550 3850 4000 3850
+Wire Wire Line
+	4000 4150 4000 4050
+$Comp
+L qomu-board:TP_SMD_0_75MM TP3
+U 1 1 5E492FD8
+P 4100 4050
+F 0 "TP3" V 4100 4000 50  0000 R CNN
+F 1 "TP_SMD_0_75MM" H 4100 3950 50  0001 C CNN
+F 2 "qomu-board-footprints:Testpoint_smd_0_75mm" H 4300 4250 60  0001 L CNN
+F 3 "" H 4300 4350 60  0001 L CNN
+	1    4100 4050
+	0    -1   -1   0
+$EndComp
+Wire Notes Line
+	4450 2300 4450 7700
+Connection ~ 5450 3200
+Wire Wire Line
+	5450 3200 5050 3200
+$Comp
+L qomu-board:TP_SMD_0_75MM TP5
+U 1 1 5E4D1EDD
+P 5450 3100
+F 0 "TP5" H 5500 3000 50  0000 R CNN
+F 1 "TP_SMD_0_75MM" H 5450 3000 50  0001 C CNN
+F 2 "qomu-board-footprints:Testpoint_smd_0_75mm" H 5650 3300 60  0001 L CNN
+F 3 "" H 5650 3400 60  0001 L CNN
+	1    5450 3100
+	-1   0    0    1
+$EndComp
+$Comp
+L qomu-board:TP_SMD_0_75MM TP4
+U 1 1 5E4EF31B
+P 5450 2750
+F 0 "TP4" H 5500 2650 50  0000 R CNN
+F 1 "TP_SMD_0_75MM" H 5450 2650 50  0001 C CNN
+F 2 "qomu-board-footprints:Testpoint_smd_0_75mm" H 5650 2950 60  0001 L CNN
+F 3 "" H 5650 3050 60  0001 L CNN
+	1    5450 2750
+	-1   0    0    1
+$EndComp
+Connection ~ 5450 2850
+Wire Wire Line
+	5450 2850 5050 2850
+$Comp
+L qomu-board:TP_SMD_0_75MM TP6
+U 1 1 5E509DA9
+P 5450 3400
+F 0 "TP6" H 5400 3300 50  0000 L CNN
+F 1 "TP_SMD_0_75MM" H 5450 3300 50  0001 C CNN
+F 2 "qomu-board-footprints:Testpoint_smd_0_75mm" H 5650 3600 60  0001 L CNN
+F 3 "" H 5650 3700 60  0001 L CNN
+	1    5450 3400
+	1    0    0    -1
+$EndComp
+Connection ~ 5450 3300
+Wire Wire Line
+	5450 3300 5050 3300
+$Comp
+L qomu-board:TP_SMD_0_75MM TP7
+U 1 1 5E52A8DA
+P 6700 2750
+F 0 "TP7" H 6750 2650 50  0000 R CNN
+F 1 "TP_SMD_0_75MM" H 6700 2650 50  0001 C CNN
+F 2 "qomu-board-footprints:Testpoint_smd_0_75mm" H 6900 2950 60  0001 L CNN
+F 3 "" H 6900 3050 60  0001 L CNN
+	1    6700 2750
+	-1   0    0    1
+$EndComp
+$Comp
+L qomu-board:TP_SMD_0_75MM TP1
+U 1 1 5E53D85B
+P 1300 3600
+F 0 "TP1" H 1350 3500 50  0000 R CNN
+F 1 "TP_SMD_0_75MM" H 1300 3500 50  0001 C CNN
+F 2 "qomu-board-footprints:Testpoint_smd_0_75mm" H 1500 3800 60  0001 L CNN
+F 3 "" H 1500 3900 60  0001 L CNN
+	1    1300 3600
+	-1   0    0    1
+$EndComp
+Connection ~ 1300 3700
+Wire Wire Line
+	1300 3700 1100 3700
+Connection ~ 6700 2850
+Wire Wire Line
+	6700 2850 7100 2850
+$Comp
+L qomu-board:TP_SMD_0_75MM TP8
+U 1 1 5E562531
+P 6750 3300
+F 0 "TP8" V 6850 3350 50  0000 R CNN
+F 1 "TP_SMD_0_75MM" H 6750 3200 50  0001 C CNN
+F 2 "qomu-board-footprints:Testpoint_smd_0_75mm" H 6950 3500 60  0001 L CNN
+F 3 "" H 6950 3600 60  0001 L CNN
+	1    6750 3300
+	0    -1   -1   0
+$EndComp
+Connection ~ 6650 3300
 $EndSCHEMATC
