File: qomu-board.sch (KiCad schematic (older format))
At the start: 60 parts, among them IC1 EOS-S3, J1 FTSH-105-01-L-DV-K, J2 825437-4, J3 22-23-2021, Q1 RV1C002UN, Q2 RV1C002UN, Q3 RV1C002UN, SW2 Captouch Pads, U1 MIC5504-3.3YMT, U10 UHD1110-FKA, U2 MIC5504-3.3YMT, U4 GD25Q16CEIGR, U5 MC3635, U9 USB-B

Commit message: Added GP testpoints, routing
Parts:
- added TP?: TP_SMD_0_75MM, qomu-board-footprints:Testpoint_smd_0_75_0_6mm, symbol qomu-board:TP_SMD_0_75MM
- TP1, TP2, TP3: footprint qomu-board-footprints:Testpoint_smd_0_75mm -> qomu-board-footprints:Testpoint_smd_0_75_0_6mm
Connections:
- wire segments 229 -> 230
Changed lines of the file:
@@
 F 0 "TP2" V 4100 3800 50  0000 R CNN
 F 1 "TP_SMD_0_75MM" H 4100 3750 50  0001 C CNN
-F 2 "qomu-board-footprints:Testpoint_smd_0_75mm" H 4300 4050 60  0001 L CNN
+F 2 "qomu-board-footprints:Testpoint_smd_0_75_0_6mm" H 4300 4050 60  0001 L CNN
 F 3 "" H 4300 4150 60  0001 L CNN
 	1    4100 3850
@@
 F 0 "TP3" V 4100 4000 50  0000 R CNN
 F 1 "TP_SMD_0_75MM" H 4100 3950 50  0001 C CNN
-F 2 "qomu-board-footprints:Testpoint_smd_0_75mm" H 4300 4250 60  0001 L CNN
+F 2 "qomu-board-footprints:Testpoint_smd_0_75_0_6mm" H 4300 4250 60  0001 L CNN
 F 3 "" H 4300 4350 60  0001 L CNN
 	1    4100 4050
@@
 F 0 "TP1" H 1350 3500 50  0000 R CNN
 F 1 "TP_SMD_0_75MM" H 1300 3500 50  0001 C CNN
-F 2 "qomu-board-footprints:Testpoint_smd_0_75mm" H 1500 3800 60  0001 L CNN
+F 2 "qomu-board-footprints:Testpoint_smd_0_75_0_6mm" H 1500 3800 60  0001 L CNN
 F 3 "" H 1500 3900 60  0001 L CNN
 	1    1300 3600
@@
 $EndComp
 Connection ~ 6650 3300
+$Comp
+L qomu-board:TP_SMD_0_75MM TP?
+U 1 1 5E5F7FB2
+P 1100 4600
+F 0 "TP?" H 1150 4500 50  0000 R CNN
+F 1 "TP_SMD_0_75MM" H 1100 4500 50  0001 C CNN
+F 2 "qomu-board-footprints:Testpoint_smd_0_75_0_6mm" H 1300 4800 60  0001 L CNN
+F 3 "" H 1300 4900 60  0001 L CNN
+	1    1100 4600
+	-1   0    0    1
+$EndComp
+Wire Wire Line
+	1100 4700 1300 4700
 $EndSCHEMATC

Commit message: Edited tech notes on PCB
Parts:
- gave numbers to parts that had none: 1
Changed lines of the file:
@@
 Connection ~ 6650 3300
 $Comp
-L qomu-board:TP_SMD_0_75MM TP?
+L qomu-board:TP_SMD_0_75MM TP9
 U 1 1 5E5F7FB2
 P 1100 4600
-F 0 "TP?" H 1150 4500 50  0000 R CNN
+F 0 "TP9" H 1150 4500 50  0000 R CNN
 F 1 "TP_SMD_0_75MM" H 1100 4500 50  0001 C CNN
 F 2 "qomu-board-footprints:Testpoint_smd_0_75_0_6mm" H 1300 4800 60  0001 L CNN
